File: GNI-plutoclocker.kicad_pcb (KiCad board)
At the start: 2 copper layers, 49 x 47 mm, 65 parts, among them J1 PLUTO_RF_IN, J2 PLUTO_5V, J3 PLUTO_40MHZ_IN, J4 10MHZ_IN, J5 LNB_OUT, J6 10MHZ_OUT, J7 I2C_PROG, J8 18V_ENA, U1 MIC5504-3.3YM5, U2 MIC5504-1.8YM5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

Commit message: adding some project changes and fab outputs
Parts:
- removed C20: 10p, Capacitor_SMD:C_0805_2012Metric
- added C12: 10u, Capacitor_SMD:C_0805_2012Metric, F.Cu at (102.8, 88.2)
- added L9: 4.7uH, Inductor_SMD:L_0805_2012Metric_Pad1.15x1.40mm_HandSolder, F.Cu at (99.5, 89.2)
- added TP1: S0_PAD, Connector_PinSocket_2.54mm:PinSocket_1x01_P2.54mm_Vertical, F.Cu at (128.2, 86.0)
- C10, C9: value 1n -> 100n
- C6: footprint Capacitor_THT:CP_Radial_D8.0mm_P3.80mm -> Capacitor_SMD:C_0805_2012Metric
- J7: footprint Connector_PinSocket_2.54mm:PinSocket_1x04_P2.54mm_Vertical -> Connector_PinSocket_2.54mm:PinSocket_1x03_P2.54mm_Vertical
- J8: footprint Inductor_SMD:L_0805_2012Metric_Pad1.15x1.40mm_HandSolder -> TestPoint:TestPoint_2Pads_Pitch2.54mm_Drill0.8mm
- L3: footprint Inductor_SMD:L_0805_2012Metric_Pad1.15x1.40mm_HandSolder -> Inductor_SMD:L_Fastron_PISN_Handsoldering
- moved C3 35.5 mm to (120.8, 71.2), turned to 180 degrees
- moved U2 31.3 mm to (120.7, 74.4), turned to 270 degrees
- moved C10 29.0 mm to (120.7, 77.5)
- moved C2 28.1 mm to (115.5, 71.2), turned to 180 degrees
- moved C17 26.5 mm to (120.7, 79.5), turned to 180 degrees
- moved U1 24.1 mm to (115.6, 74.4), turned to 270 degrees
- moved C23 23.5 mm to (95.6, 74.0), turned to 300 degrees
- moved C9 22.7 mm to (115.5, 77.5)
- moved C6 22.3 mm to (97.8, 85.5), turned to 0 degrees
- moved J3 20.4 mm to (103.0, 95.0), turned to 0 degrees
- moved R2 19.6 mm to (105.5, 92.1)
- moved C16 19.6 mm to (115.5, 79.5), turned to 180 degrees
- moved C4 19.6 mm to (108.5, 92.8)
- moved R9 18.3 mm to (115.3, 67.5), turned to 0 degrees
- moved C25 17.8 mm to (115.3, 65.5), turned to 180 degrees
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Connections:
- C2 pad 1: +5V -> Net-(C12-Pad1)
- C3 pad 1: +5V -> Net-(C12-Pad1)
- J7 pad 3: Net-(J7-Pad3) -> GND
- R16 pad 2: Net-(J7-Pad2) -> Net-(J7-Pad1)
- R17 pad 2: Net-(J7-Pad3) -> Net-(J7-Pad2)
- U1 pad 1: +5V -> Net-(C12-Pad1)
- U1 pad 3: +5V -> Net-(C12-Pad1)
- U2 pad 1: +5V -> Net-(C12-Pad1)
- U2 pad 3: +5V -> Net-(C12-Pad1)
- U4 pad 12: Net-(J7-Pad3) -> Net-(J7-Pad2)
- U4 pad 13: Net-(J7-Pad2) -> Net-(J7-Pad1)
- U4 pad 2: Net-(J7-Pad1) -> Net-(TP1-Pad1)
Routing:
- net GND: track 0.00 -> 99.0 mm, vias 0 -> 31
- net Net-(C12-Pad1): track 0.00 -> 59.3 mm, vias 0 -> 2
- net +3V3: track 0.00 -> 34.5 mm, vias 0 -> 3
- net Net-(C22-Pad1): track 0.00 -> 32.8 mm, vias 0 -> 1
- net +1V8: track 0.00 -> 31.4 mm
- net +5V: track 0.00 -> 28.1 mm, vias 0 -> 2
- net Net-(C25-Pad1): track 0.00 -> 24.7 mm
- net Net-(D1-Pad2): track 0.00 -> 17.0 mm
- net Net-(C15-Pad1): track 0.00 -> 9.86 mm, vias 0 -> 2
- net Net-(C25-Pad2): track 0.00 -> 9.19 mm
- net Net-(TP1-Pad1): track 0.00 -> 8.90 mm
- net Net-(C29-Pad1): track 0.00 -> 7.80 mm
- net Net-(J1-Pad1): track 0.00 -> 7.77 mm
- net Net-(R11-Pad1): track 0.00 -> 6.71 mm
- net Net-(C21-Pad1): track 0.00 -> 6.51 mm
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- added copper zone on F.Cu, net +5V
- added copper zone on B.Cu, net GND
- added copper zone on F.Cu, net GND
- added copper zone on F.Cu, net Net-(C22-Pad1)
- added copper zone on F.Cu, net Net-(D1-Pad2)
Other:
- rule pad_to_mask_clearance: 0.05 -> 0

Commit message: minor aesthetics schematics and silk layer adjustments
Other:
- board text added: "(G)"
- board text added: "GNI-plutoclocker rev. 1.0 (C) SP5GNI + SO5UCC"
- board text added: "github.com/cr1tbit/GNI-plutoclocker"
